Commit message: Add link coloring

File: urdf/16ton_macro.xacro (robot description, xacro)
@@ -2,8 +2,20 @@
 <robot xmlns:xacro="http://ros.org/wiki/xacro">
 <xacro:macro name="coaliron_16ton" params="prefix">
+    <!-- Color Macros -->
+    <xacro:macro name="material_coaliron_grey">
+        <material name="">
+            <color rgba="0.5 0.55 0.9 1"/>
+        </material>
+    </xacro:macro>
+    <xacro:macro name="material_coaliron_head">
+        <material name="">
+            <color rgba="0.5 0.55 0.9 0.8"/>
+        </material>
+    </xacro:macro>
     <!-- link list -->
     <link name="${prefix}base_link">
         <visual>
             <origin xyz="0 0 0" rpy="0 0 0"/>
+            <xacro:material_coaliron_grey />
             <geometry>
                 <mesh filename="package://coaliron_16ton_support/meshes/visual/base_link_visual.stl" />
@@ -21,4 +33,5 @@
         <visual>
             <origin xyz="0 0 0" rpy="0 0 0"/>
+            <xacro:material_coaliron_head />
             <geometry>
                 <mesh filename="package://coaliron_16ton_support/meshes/visual/upper_mount_visual.stl"/>
@@ -30,7 +43,4 @@
                 <mesh filename="package://coaliron_16ton_support/meshes/collision/upper_mount_collision.stl"/>
             </geometry>
-            <material>
-                <color rgba="0.5 0.55 0.9 0.8"/>
-            </material>
         </collision>
     </link>
