Commit message: Add Coaliron Press URDF (#14)
* Coaliron press urdf, published 12-22-22

* Resolved notes from PR review.

* Updates collision and visual meshes to match

* Add link coloring

* Removed internal geometry from collision meshes

Simplified collision meshes by removing internal geometry and cutting down the number of vertices/faces.

* Set versioning

* add CMakeLists folder inclusions
* update package.xml version to match repo & control code version
* Add Tal to authors list

---------

Co-authored-by: acbuynak <44533530+acbuynak@users.noreply.github.com>

File: urdf/16ton.xacro (robot description, xacro)
@@ -1,2 +1,3 @@
+<?xml version="1.0" ?>
 <robot name="coaliron_16ton" xmlns:xacro="http://ros.org/wiki/xacro">
 	<xacro:include filename="$(find coaliron_16ton_support)/urdf/16ton_macro.xacro" />

File: urdf/16ton_macro.xacro (robot description, xacro)
@@ -2,10 +2,22 @@
 <robot xmlns:xacro="http://ros.org/wiki/xacro">
 <xacro:macro name="coaliron_16ton" params="prefix">
+    <!-- Color Macros -->
+    <xacro:macro name="material_coaliron_grey">
+        <material name="">
+            <color rgba="0.5 0.55 0.9 1"/>
+        </material>
+    </xacro:macro>
+    <xacro:macro name="material_coaliron_head">
+        <material name="">
+            <color rgba="0.5 0.55 0.9 0.8"/>
+        </material>
+    </xacro:macro>
     <!-- link list -->
-    <link name="${prefix}link_0">
+    <link name="${prefix}base_link">
         <visual>
             <origin xyz="0 0 0" rpy="0 0 0"/>
+            <xacro:material_coaliron_grey />
             <geometry>
-                <box size="0.1 0.3 0.1" />
+                <mesh filename="package://coaliron_16ton_support/meshes/visual/base_link_visual.stl" />
             </geometry>
         </visual>
@@ -13,13 +25,15 @@
             <origin xyz="0 0 0" rpy="0 0 0"/>
             <geometry>
-                <box size="0.1 0.3 0.1" />
+                <mesh filename="package://coaliron_16ton_support/meshes/collision/base_link_collision.stl" />
             </geometry>
         </collision>
     </link>
-    <link name="${prefix}link_1">
+    <!-- upper_mount is the moving part of the press -->
+    <link name="${prefix}upper_mount">
         <visual>
             <origin xyz="0 0 0" rpy="0 0 0"/>
+            <xacro:material_coaliron_head />
             <geometry>
-                <box size="0.1 0.3 0.1" />
+                <mesh filename="package://coaliron_16ton_support/meshes/visual/upper_mount_visual.stl"/>
             </geometry>
         </visual>
@@ -27,18 +41,39 @@
             <origin xyz="0 0 0" rpy="0 0 0"/>
             <geometry>
-                <box size="0.1 0.3 0.1" />
+                <mesh filename="package://coaliron_16ton_support/meshes/collision/upper_mount_collision.stl"/>
             </geometry>
         </collision>
     </link>
     <!-- end of link list -->
-    <!-- joint list -->
-    <joint name="${prefix}joint_1" type="prismatic">
-        <parent link="${prefix}link_0"/>
-        <child link="${prefix}link_1"/>
-        <origin xyz="0 0 0" rpy="0 0 0" />
-        <axis xyz="0 0 -1" />
-        <limit lower="0" upper="0.1524" effort="100" velocity="10"/>
-    </joint>
-    <!-- end of joint list -->
+<!-- joint list -->
+<!--base_fc (front-center) to base_link transform-->
+<link name="${prefix}base_fc" />
+<joint name="${prefix}base_fc_to_base_link" type="fixed">
+    <parent link="${prefix}base_fc"/>
+    <child link="${prefix}base_link"/>
+    <origin xyz="0 0.41046 -0.103124" rpy="0 0 0"/>
+</joint>
+<!--base_link to press_frame transform-->
+<link name="${prefix}press_frame" />
+<joint name="${prefix}base_to_press" type="fixed">
+    <parent link="${prefix}base_link"/>
+    <child link="${prefix}press_frame"/>
+    <origin xyz="0.130302 0.001524 1.5113" rpy="0 0 0"/>
+</joint>
+<!--press_frame to upper_mount transform-->
+<joint name="${prefix}moving_joint" type="prismatic">
+    <parent link="${prefix}press_frame"/>
+    <child link="${prefix}upper_mount"/>
+    <origin xyz="0.00127 -0.001524 -0.20955" rpy="0 0 0" />
+    <axis xyz="0 0 -1" />
+    <limit lower="0" upper="0.28575" effort="100" velocity="10"/>
+</joint>
+<!--base_link to lower_mount transform-->
+<link name="${prefix}lower_mount" />
+<joint name="${prefix}base_to_lower_mount" type="fixed">
+    <parent link="${prefix}base_link"/>
+    <child link="${prefix}lower_mount"/>
+    <origin xyz="0.129032 0 1.016" rpy="0 0 0"/>
+</joint>
     </xacro:macro>
 </robot>
